File: PCB/PCB.kicad_pcb (KiCad board)
At the start: 2 copper layers, 302 x 20 mm, 14 parts

Commit message: more
Parts:
- added C1: 1uF, Capacitor_SMD:C_0402_1005Metric, F.Cu at (261.0, 75.0)
- added C10: 1uF, Capacitor_SMD:C_0402_1005Metric, F.Cu at (257.8, 74.3)
- added C11: 0.1uF, Capacitor_SMD:C_0402_1005Metric, F.Cu at (258.7, 74.3)
- added C12: 0.1uF, Capacitor_SMD:C_0402_1005Metric, F.Cu at (259.8, 74.3)
- added C13: 10uF, Capacitor_SMD:C_0402_1005Metric, F.Cu at (291.2, 74.8)
- added C14: 10uF, Capacitor_SMD:C_0402_1005Metric, F.Cu at (292.5, 74.8)
- added C15: 33pF, Capacitor_SMD:C_0402_1005Metric, F.Cu at (289.9, 89.5)
- added C16: 33pF, Capacitor_SMD:C_0402_1005Metric, F.Cu at (290.1, 84.0)
- added C17: 0.1uF, Capacitor_SMD:C_0402_1005Metric, F.Cu at (275.0, 86.6)
- added C2: 0.1uF, Capacitor_SMD:C_0402_1005Metric, F.Cu at (262.2, 75.8)
- added C3: 0.1uF, Capacitor_SMD:C_0402_1005Metric, F.Cu at (263.5, 76.5)
- added C4: 0.1uF, Capacitor_SMD:C_0402_1005Metric, F.Cu at (262.2, 78.0)
- added C5: 0.1uF, Capacitor_SMD:C_0402_1005Metric, F.Cu at (263.8, 78.5)
- added C6: 0.1uF, Capacitor_SMD:C_0402_1005Metric, F.Cu at (262.5, 80.3)
- added C7: 0.1uF, Capacitor_SMD:C_0402_1005Metric, F.Cu at (264.0, 74.5)
- added C8: 0.1uF, Capacitor_SMD:C_0402_1005Metric, F.Cu at (262.2, 73.3)
- added C9: 0.1uF, Capacitor_SMD:C_0402_1005Metric, F.Cu at (264.0, 80.8)
- added J1: USB_C_Receptacle_USB2.0_14P, Connector_USB:USB_C_Receptacle_HRO_TYPE-C-31-M-12, F.Cu at (299.7, 85.7)
- added J2: Conn_01x20, Library:20_SMD, F.Cu at (269.7, 89.7)
- added J3: Conn_01x20, Library:20_SMD, F.Cu at (248.7, 89.7)
- added J4: Conn_01x03, Library:3_SMD, F.Cu at (275.6, 89.8)
- added R1: 5.1K, Resistor_SMD:R_0402_1005Metric, F.Cu at (272.8, 73.7)
- added R2: 5.1K, Resistor_SMD:R_0402_1005Metric, F.Cu at (276.3, 73.7)
- added R3: 27, Resistor_SMD:R_0402_1005Metric, F.Cu at (279.0, 73.7)
- added R4: 27, Resistor_SMD:R_0402_1005Metric, F.Cu at (281.3, 73.7)
- added R5: 1K, Resistor_SMD:R_0402_1005Metric, F.Cu at (287.6, 87.0)
- added R6: 10K, Resistor_SMD:R_0402_1005Metric, F.Cu at (283.3, 73.7)
- added R7: 1K, Resistor_SMD:R_0402_1005Metric, F.Cu at (286.0, 73.9)
- added SW1: SW_Push, Button_Switch_SMD:SW_Push_SPST_NO_Alps_SKRK, F.Cu at (270.1, 85.8)
- added U1: RP2040, Package_DFN_QFN:QFN-56-1EP_7x7mm_P0.4mm_EP3.2x3.2mm, F.Cu at (282.7, 86.2)
- added U2: W25Q16JVUXIQ TR, Package_SON:Winbond_USON-8-1EP_3x2mm_P0.5mm_EP0.2x1.6mm, F.Cu at (276.8, 86.5)
- added U4: MCP1700x-330xxTT, Package_TO_SOT_SMD:SOT-23, F.Cu at (292.8, 82.5)
- added Y1: 12 MHz, Crystal:Crystal_SMD_3225-4Pin_3.2x2.5mm, F.Cu at (289.9, 86.8)
Routing:
- net QSPI_SS: track 0.00 -> 8.27 mm
- net QSPI_SD1: track 0.00 -> 6.51 mm
- net QSPI_SD2: track 0.00 -> 4.77 mm
Other:
- board text removed: "3.14159265358979323846264338327950288419716939937510 58209749445923078164062862089986280348253421170679"

Commit message: s
Routing:
- net QSPI_SD0: track 0.00 -> 6.74 mm
- net QSPI_SCLK: track 0.00 -> 4.92 mm
Changed lines of the file:
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@@
+	)
+	(segment
+		(start 275.649 86.2)
+		(end 275.649 87.037798)
+		(width 0.2)
+		(layer "F.Cu")
+		(net 48)
+	)
+	(segment
+		(start 277.5 85.075)
+		(end 277.5 85.540798)
+		(width 0.2)
+		(layer "F.Cu")
+		(net 48)
+	)
+	(segment
+		(start 278.138798 87.598)
+		(end 278.725226 87.598)
+		(width 0.2)
+		(layer "F.Cu")
+		(net 48)
+	)
+	(segment
+		(start 277.5 85.540798)
+		(end 276.941798 86.099)
+		(width 0.2)
+		(layer "F.Cu")
+		(net 48)
+	)
+	(segment
+		(start 277.714798 87.174)
+		(end 278.138798 87.598)
+		(width 0.2)
+		(layer "F.Cu")
+		(net 48)
+	)
+	(segment
+		(start 275.785202 87.174)
+		(end 277.714798 87.174)
+		(width 0.2)
+		(layer "F.Cu")
+		(net 48)
+	)
+	(segment
+		(start 275.75 86.099)
+		(end 275.649 86.2)
+		(width 0.2)
+		(layer "F.Cu")
+		(net 48)
+	)
+	(segment
+		(start 276.941798 86.099)
+		(end 275.75 86.099)
+		(width 0.2)
+		(layer "F.Cu")
+		(net 48)
+	)
+	(segment
+		(start 275.649 87.037798)
+		(end 275.785202 87.174)
+		(width 0.2)
+		(layer "F.Cu")
+		(net 48)
 	)
 	(segment
@@
 		(net 52)
 	)
+	(segment
+		(start 277.851 86.773)
+		(end 277.926 86.698)
+		(width 0.2)
+		(layer "F.Cu")
+		(net 53)
+	)
+	(segment
+		(start 277 84.609202)
+		(end 277.285202 84.324)
+		(width 0.2)
+		(layer "F.Cu")
+		(net 53)
+	)
+	(segment
+		(start 277.714798 84.324)
+		(end 277.926 84.535202)
+		(width 0.2)
+		(layer "F.Cu")
+		(net 53)
+	)
+	(segment
+		(start 277.926 84.535202)
+		(end 277.926 86.698)
+		(width 0.2)
+		(layer "F.Cu")
+		(net 53)
+	)
+	(segment
+		(start 277.851 86.773)
+		(end 277.880898 86.773)
+		(width 0.2)
+		(layer "F.Cu")
+		(net 53)
+	)
+	(segment
+		(start 277 85.075)
+		(end 277 84.609202)
+		(width 0.2)
+		(layer "F.Cu")
+		(net 53)
+	)
+	(segment
+		(start 277.285202 84.324)
+		(end 277.714798 84.324)
+		(width 0.2)
+		(layer "F.Cu")
+		(net 53)
+	)
+	(segment
+		(start 278.304898 87.197)
+		(end 278.724226 87.197)
+		(width 0.2)
+		(layer "F.Cu")
+		(net 53)
+	)
+	(segment
+		(start 277.880898 86.773)
+		(end 278.304898 87.197)
+		(width 0.2)
+		(layer "F.Cu")
+		(net 53)
+	)
 	(embedded_fonts no)
